Commit message: Added wheel and inertial property

File: description/robot_core.xacro (robot description, xacro)
@@ -1,4 +1,6 @@
 <?xml version="1.0"?>
 <robot xmlns:xacro="http://www.ros.org/wiki/xacro" >
+    <xacro:include filename="inertial_macros.xacro"/>
+    <!-- Define material property-->
     <material name="white">
         <color rgba="1 1 1 1"/>
@@ -13,4 +15,5 @@
         <color rgba="0 0 0 1"/>
     </material>
+    <!-- Base link-->
     <link name="base_link">
     </link>
@@ -20,4 +23,5 @@
         <origin xyz="-0.1 0 0"/>
     </joint>
+    <!-- Chassis-->
     <link name="chassis">
         <visual>
@@ -28,4 +32,59 @@
             </geometry>
         </visual>
+        <xacro:inertial_box x="0.3" y="0.3" z="0.15" mass="0.7">
+            <origin xyz="0.15 0 0.075" rpy="0 0 0"/>
+        </xacro:inertial_box>
+    </link>
+    <!-- Wheel-->
+    <joint name="left_wheel_joint" type="continuous">
+        <parent link="base_link"/>
+        <child link="left_wheel"/>
+        <origin xyz="0 0.175 0" rpy="-${pi/2} 0 0"/>
+        <axis xyz="0 0 1"/>
+    </joint>
+    <link name="left_wheel">
+        <visual>
+            <material name="blue"/>
+            <geometry>
+                <cylinder radius="0.05" length="0.04"/>
+            </geometry>
+        </visual>
+        <xacro:inertial_cylinder radius="0.05" length="0.04" mass="0.3">
+            <origin xyz="0 0 0" rpy="0 0 0"/>
+        </xacro:inertial_cylinder>
+    </link>
+    <joint name="right_wheel_joint" type="continuous">
+        <parent link="base_link"/>
+        <child link="right_wheel"/>
+        <origin xyz="0 -0.175 0" rpy="${pi/2} 0 0"/>
+        <axis xyz="0 0 -1"/>
+    </joint>
+    <link name="right_wheel">
+        <visual>
+            <material name="blue"/>
+            <geometry>
+                <cylinder radius="0.05" length="0.04"/>
+            </geometry>
+        </visual>
+        <xacro:inertial_cylinder radius="0.05" length="0.04" mass="0.3">
+            <origin xyz="0 0 0" rpy="0 0 0"/>
+        </xacro:inertial_cylinder>
+    </link>
+    <!-- Caster wheel-->
+    <joint name="caster_joint" type="fixed">
+        <parent link="base_link"/>
+        <child link="caster_wheel"/>
+        <origin xyz="0.1 0 0"/>
+    </joint>
+    <link name="caster_wheel">
+        <visual>
+            <material name="black"/>
+            <geometry>
+                <sphere radius="0.05"/>
+            </geometry>
+        </visual>
+        <xacro:inertial_sphere radius="0.05" mass="0.2">
+            <origin xyz="0 0 0" rpy="0 0 0"/>
+        </xacro:inertial_sphere>
     </link>
 </robot>

Commit message: Added gazebo property in xacro and created new launch file

File: description/robot_core.xacro (robot description, xacro)
@@ -36,4 +36,7 @@
         </xacro:inertial_box>
     </link>
+    <gazebo reference="chassis">
+        <material>Gazebo/White</material>
+    </gazebo>
     <!-- Wheel-->
     <joint name="left_wheel_joint" type="continuous">
@@ -54,4 +57,7 @@
         </xacro:inertial_cylinder>
     </link>
+    <gazebo reference="left_wheel">
+    <material>Gazebo/Blue</material>
+    </gazebo>
     <joint name="right_wheel_joint" type="continuous">
         <parent link="base_link"/>
@@ -71,4 +77,7 @@
         </xacro:inertial_cylinder>
     </link>
+    <gazebo reference="right_wheel">
+    <material>Gazebo/Blue</material>
+    </gazebo>
     <!-- Caster wheel-->
     <joint name="caster_joint" type="fixed">
@@ -88,3 +97,8 @@
         </xacro:inertial_sphere>
     </link>
+    <gazebo reference="caster_wheel">
+        <material>Gazebo/Black</material>
+        <mu1 value="0.0001"/>
+        <mu2 value="0.0001"/>
+    </gazebo>
 </robot>
