Commit message: laser sacnner added

File: description/gazebo_control.xacro (robot description, xacro)
@@ -2,14 +2,14 @@
 <robot xmlns:xacro="http://www.ros.org/wiki/xacro">
     <gazebo>
-        <!-- Wheel information-->
-        <plugin name ="diff_drive" filename="libgazebo_ros_diff_drive.so">
+        <plugin name='diff_drive' filename='libgazebo_ros_diff_drive.so'>
+            <!-- Wheel Information -->
             <left_joint>left_wheel_joint</left_joint>
             <right_joint>right_wheel_joint</right_joint>
-            <wheel_seperation>0.35</wheel_seperation>
+            <wheel_separation>0.35</wheel_separation>
             <wheel_diameter>0.1</wheel_diameter>
-            <!-- limits-->
+            <!-- Limits -->
             <max_wheel_torque>200</max_wheel_torque>
-            <max_wheel_acceleration>10</max_wheel_acceleration>
-            <!-- output-->
+            <max_wheel_acceleration>10.0</max_wheel_acceleration>
+            <!-- Output -->
             <odometry_frame>odom</odometry_frame>
             <robot_base_frame>base_link</robot_base_frame>

File: description/robot.urdf.xacro (robot description, xacro)
@@ -3,3 +3,5 @@
     <xacro:include filename="robot_core.xacro"/>
     <xacro:include filename="wheel_control.xacro"/>
+    <xacro:include filename="gazebo_control.xacro"/>
+    <xacro:include filename="laser.xacro"/>
 </robot>

File: description/robot_core.xacro (robot description, xacro)
@@ -32,4 +32,10 @@
             </geometry>
         </visual>
+        <collision>
+            <origin xyz="0.15 0 0.075"/>
+            <geometry>
+                <box size="0.3 0.3 0.15"/>
+            </geometry>
+        </collision>
         <xacro:inertial_box x="0.3" y="0.3" z="0.15" mass="0.7">
             <origin xyz="0.15 0 0.075" rpy="0 0 0"/>
@@ -53,4 +59,9 @@
             </geometry>
         </visual>
+        <collision>
+            <geometry>
+                <cylinder radius="0.05" length="0.04"/>
+            </geometry>
+        </collision>
         <xacro:inertial_cylinder radius="0.05" length="0.04" mass="0.3">
             <origin xyz="0 0 0" rpy="0 0 0"/>
@@ -73,4 +84,9 @@
             </geometry>
         </visual>
+        <collision>
+            <geometry>
+                <cylinder radius="0.05" length="0.04"/>
+            </geometry>
+        </collision>
         <xacro:inertial_cylinder radius="0.05" length="0.04" mass="0.3">
             <origin xyz="0 0 0" rpy="0 0 0"/>
@@ -93,4 +109,9 @@
             </geometry>
         </visual>
+        <collision>
+            <geometry>
+                <sphere radius="0.05"/>
+            </geometry>
+        </collision>
         <xacro:inertial_sphere radius="0.05" mass="0.2">
             <origin xyz="0 0 0" rpy="0 0 0"/>
