Commit message: laser bug fixed

File: description/laser.xacro (robot description, xacro)
@@ -1,2 +1,3 @@
+<?xml version="1.0"?>
 <robot xmlns:xacro="http://www.ros.org/wiki/xacro">
     <xacro:include filename="inertial_macros.xacro"/>
@@ -7,5 +8,5 @@
         <parent link="base_link"/>
         <child link="laser"/>
-        <origin xyz="0.13 0 0.15"/>
+        <origin xyz="0.13 0 0.165"/>
     </joint>
     <link name="laser">
@@ -21,9 +22,7 @@
             </geometry>
         </collision>
-        <inertial>
-            <xacro:inertial_cylinder radius="0.05" length="0.03" mass="1.0">
+        <xacro:inertial_cylinder radius="0.05" length="0.03" mass="1.0">
                 <origin xyz="0 0 0" rpy="0 0 0"/>
-            </xacro:inertial_cylinder>
-        </inertial>
+        </xacro:inertial_cylinder>
     </link>
     <gazebo reference="laser">

File: description/wheel_control.xacro (robot description, xacro)
@@ -6,5 +6,5 @@
             <left_joint>left_wheel_joint</left_joint>
             <right_joint>right_wheel_joint</right_joint>
-            <wheel_seperation>0.35</wheel_seperation>
+            <wheel_separation>0.35</wheel_separation>
             <wheel_diameter>0.1</wheel_diameter>
             <!-- limits-->

Commit message: laser scan bug fixed

File: description/laser.xacro (robot description, xacro)
@@ -8,5 +8,5 @@
         <parent link="base_link"/>
         <child link="laser"/>
-        <origin xyz="0.13 0 0.165"/>
+        <origin xyz="0.13 0 0.2"/>
     </joint>
     <link name="laser">
@@ -41,6 +41,6 @@
                 </scan>
                 <range>
-                    <min>0.02</min>
-                    <max>5</max>
+                    <min>0.08</min>
+                    <max>10</max>
                 </range>
             </ray>

File: description/robot.urdf.xacro (robot description, xacro)
@@ -3,5 +3,4 @@
     <xacro:include filename="robot_core.xacro"/>
     <xacro:include filename="wheel_control.xacro"/>
-    <xacro:include filename="gazebo_control.xacro"/>
     <xacro:include filename="laser.xacro"/>
 </robot>

File: description/robot_core.xacro (robot description, xacro)
@@ -17,4 +17,5 @@
     <!-- Base link-->
     <link name="base_link">
+        <origin xyz="0 0 100"/>
     </link>
     <joint name="chassis_joint" type="fixed">
